File: acmi-pwrbrd.kicad_sch (KiCad schematic)
At the start: 25 parts, among them J1 430450402, J10 3-641215-8, J2 430450402, J3 430451202, J4 430451202, J5 430450402

Commit message: Finish routing
Parts:
- removed J10: 3-641215-8, 3-641215-8:TE_3-641215-8, symbol myparts:3-641215-8
- added J6: 39289108, myparts:MOLEX_39289108, symbol myparts:39289108
- added J7: 430451202, myparts:CONN_SD-43045-001_12_MOL, symbol myparts:430451202
Connections:
- net +12V: now also J6.1
- net +15V: now also J6.2, J7.1, J7.7
- net +5V: now also J6.4, J7.2, J7.8
- net -15V: now also J6.3, J7.12, J7.6
- net -5V: now also J6.5, J7.11, J7.5
- net GND: now also J6.10, J6.6, J6.7, J6.8, J6.9, J7.10, J7.3, J7.4, J7.9
Other:
- moved on the sheet: D1, D2, D3, D4, D5, J1, J2, J3, J4, J5, R1, R2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

Commit message: Added 12VB, testpoints, cable harness
Parts:
- removed J3: 430451202, myparts:CONN_SD-43045-001_12_MOL, symbol myparts:430451202
- removed J6: 39289108, myparts:MOLEX_39289108, symbol myparts:39289108
- added D6: ~, LED_SMD:LED_0805_2012Metric, symbol myparts:LED-0805
- added J100: RT001412SNH, symbol myparts:RT001412SNH
- added J101: 39012105, myparts:MOLEX_39289108, symbol myparts:39012105
- added J6: 39289108, myparts:MOLEX_39289108, symbol myparts:39289108-2
- added J7: 430451202, myparts:CONN_SD-43045-001_12_MOL, symbol myparts:430451202
- added N100: RC16M23K, symbol Mechanical:Housing
- added N101: 39000077, symbol Mechanical:Housing
- added R6: 895, Resistor_SMD:R_0603_1608Metric, symbol Device:R_US
- added TP6, TP7: ${SHORT_NET_NAME(1)}, TestPoint:TestPoint_Keystone_5005-5009_Compact, symbol Connector:TestPoint
- TP1, TP2, TP3, TP4, TP5: footprint TestPoint:TestPoint_THTPad_D2.0mm_Drill1.0mm -> TestPoint:TestPoint_Keystone_5005-5009_Compact
- renumbered D3 to D1, D1 to D2, D2 to D3, J5 to J1, J7 to J3, J1 to J5, R2 to R1, R1 to R2
Connections:
- net +15V: now also J6.3, J7.1, J7.7
- net +5V: now also J6.5, J7.2, J7.8
- net -15V: now also J6.4, J7.12, J7.6
- net -5V: now also J6.6, J7.11, J7.5
- net GND: now also D6.1 (K), J6.10, J6.7, J6.8, J6.9, J7.10, J7.3, J7.4, J7.9, TP7.1
- net +12V renamed +12VA
- net +12VA: now also J6.1; no longer J2.1
- new net: D6.2 (A), R6.2
- new net +12VA_OUT: J100.D, J101.1
- new net +12VB: J2.1, J6.2, R6.1, TP6.1
- new net +12VB_OUT: J100.F, J101.2
- new net +15V_OUT: J100.A, J101.3
- new net +5V_OUT: J100.H, J101.5
- new net -15V_OUT: J100.C, J101.4
- new net -5V_OUT: J100.K, J101.6
- new net 12VA_RET_OUT: J100.E, J101.7
- new net 12VB_RET_OUT: J100.G, J101.8
- new net 15V_RET_OUT: J100.B, J101.9
- new net 5V_RET_OUT: J100.J, J101.10
- new net GNDPWR: J100.M
- no-connect marks 0 -> 4
Other:
- note added: "All conductors are to be 16AWG"
- note removed: "ACMI Power Distribution Board"
- title: (none) -> ACMI-II Power Distribution Board
- moved on the sheet: D1, D2, D3, D4, D5, MT1, MT2, MT3, MT4, R1, R2, R3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
